Commit message: added tail and readme modifications

File: urdf/robot2.xacro (robot description, xacro)
@@ -97,5 +97,5 @@
   	  <origin xyz="0 0 0" rpy="0 0 0"/>
       <geometry>
-        <box size="0.1 0.1 0.1"/>
+       <cylinder radius="0.04" length="0.20"/>
       </geometry>
   	</collision>
@@ -110,7 +110,59 @@
   </link>
   <joint name="arm_base_to_base" type="fixed">
-  	<origin rpy="0 0 0" xyz="0.20 0 0.15"/>
+  	<origin rpy="0 0 0" xyz="0.20 0 0.1"/>
   	<parent link="base_link"/>
   	<child link="arm_base_link"/>
+  </joint>
+  <link name="tail_link1">
+  	<inertial>
+  		<mass value="0.1"/>
+  		<origin xyz="0 0 0" rpy="0 0 0" />
+  		<inertia ixx="0.0000416666667" ixy="0" ixz="0" iyy="0.0000416666667" iyz="0" izz="0.0000416666667"/>
+  	</inertial>
+  	<collision>
+  	  <origin xyz="0 0 0" rpy="0 0 0"/>
+      <geometry>
+        <cylinder radius="0.04" length="0.20"/>
+      </geometry>
+  	</collision>
+  	<visual>
+  	  <origin xyz="0 0 0" rpy="0 0 0"/>
+      <geometry>
+        <!-- <box size="0.1 0.1 0.1"/> -->
+        <cylinder radius="0.02" length="0.20"/>
+      </geometry>
+      <material name="blue" />
+  	</visual>
+  </link>
+  <joint name="tail1" type="fixed">
+  	<origin rpy="0 -0.78 0" xyz="-0.20 0 0.1"/>
+  	<parent link="base_link"/>
+  	<child link="tail_link1"/>
+  </joint>
+    <link name="tail_link2">
+  	<inertial>
+  		<mass value="0.1"/>
+  		<origin xyz="0 0 0" rpy="0 0 0" />
+  		<inertia ixx="0.0000416666667" ixy="0" ixz="0" iyy="0.0000416666667" iyz="0" izz="0.0000416666667"/>
+  	</inertial>
+  	<collision>
+  	  <origin xyz="0 0 0" rpy="0 0 0"/>
+      <geometry>
+        <cylinder radius="0.02" length="0.23"/>
+      </geometry>
+  	</collision>
+  	<visual>
+  	  <origin xyz="0 0 0" rpy="0 0 0"/>
+      <geometry>
+        <!-- <box size="0.1 0.1 0.1"/> -->
+        <cylinder radius="0.02" length="0.23"/>
+      </geometry>
+      <material name="blue" />
+  	</visual>
+  </link>
+  <joint name="tail2" type="fixed">
+  	<origin xyz="-0.1 0 0.1" rpy="0 -1.56 0"/>
+  	<parent link="tail_link1"/>
+  	<child link="tail_link2"/>
   </joint>
   <link name="arm_link_01">
@@ -157,5 +209,5 @@
   	<axis xyz="1 0 0"/>
   	<limit effort="1000.0" lower="-0.78" upper="0.78" velocity="0.2"/>
-  	<origin rpy="0 0 0" xyz="0 0 0.15"/>
+  	<origin rpy="0 0 0" xyz="0 0 0.14"/>
   	<parent link="arm_base_link"/>
   	<child link="arm_link_01"/>

Commit message: color robot

File: urdf/robot2.xacro (robot description, xacro)
@@ -132,5 +132,5 @@
         <cylinder radius="0.02" length="0.20"/>
       </geometry>
-      <material name="blue" />
+      <material name="red" />
   	</visual>
   </link>
@@ -158,5 +158,5 @@
         <cylinder radius="0.02" length="0.23"/>
       </geometry>
-      <material name="blue" />
+      <material name="red" />
   	</visual>
   </link>
